Commit message: 完成建模、属性、惯性

File: robot/src/cerbers/urdf/cerbers/base.urdf.xacro (robot description, xacro)
@@ -1,5 +1,7 @@
 <?xml version="1.0"?>
 <robot xmlns:xacro="http://www.ros.org/wiki/xacro">
+<xacro:include filename="$(find cerbers)/urdf/cerbers/common_inertial.xacro"/>
     <xacro:macro name="base_xacro" params="length radius">
+        <link name="base_footprint" />
         <link name="base_link">
             <!-- 部件外观描述 -->
@@ -17,5 +19,24 @@
                 </material>
             </visual>
+            <collision>
+                <!-- 沿着自己几何中心的偏移和旋转 -->
+                <origin xyz="0.0 0.0 0.0" rpy="0.0 0.0 0.0"/>
+                <!-- 几何形状 -->
+                <geometry>
+                    <!-- 圆柱体 radius半径，length高度 -->
+                    <cylinder radius="${radius}" length="${length}"/>
+                </geometry>
+                <!-- 材质描述 -->
+                <material name="white">
+                    <color rgba="1.0 1.0 1.0 0.5"/>
+                </material>
+            </collision>
+        <xacro:cylinder_inertia m="1.0" r="${radius}" h="${length}" />
         </link>
+        <joint name="joint_name" type="fixed">
+            <origin xyz="0.0 0.0 ${length/2+0.032-0.001}" rpy="0.0 0.0 0.0"/>
+            <parent link="base_footprint"/>
+            <child link="base_link"/>
+        </joint>
     </xacro:macro>
 </robot>

File: robot/src/cerbers/urdf/cerbers/cerbers.urdf.xacro (robot description, xacro)
@@ -7,4 +7,7 @@
 <xacro:include filename="sensor/camera.urdf.xacro"/>
 <xacro:include filename="sensor/laser.urdf.xacro"/>
+<!-- 执行器 -->
+<xacro:include filename="actuator/wheel.urdf.xacro"/>
+<xacro:include filename="actuator/caster.urdf.xacro"/>
 <!-- 调用宏 -->
 <xacro:base_xacro length="0.12" radius="0.1" />
@@ -12,3 +15,7 @@
 <xacro:camera_xacro xyz="0.10 0.0 0.075" />
 <xacro:laser_xacro xyz="0.0 0.0 0.11" />
+<xacro:wheel_xacro wheel_name="left_wheel" xyz="0.0 0.10 -0.06" />
+<xacro:wheel_xacro wheel_name="right_wheel" xyz="0.0 -0.10 -0.06" />
+<xacro:caster_xacro caster_name="front_caster" xyz="0.08 0.0 -0.076" />
+<xacro:caster_xacro caster_name="back_caster" xyz="-0.08 0.0 -0.076" />
 </robot>

File: robot/src/cerbers/urdf/cerbers/sensor/camera.urdf.xacro (robot description, xacro)
@@ -1,4 +1,5 @@
 <?xml version="1.0"?>
 <robot xmlns:xacro="http://www.ros.org/wiki/xacro">
+<xacro:include filename="$(find cerbers)/urdf/cerbers/common_inertial.xacro"/>
     <xacro:macro name="camera_xacro" params="xyz">
         <!-- 机器人的camera-->
@@ -17,4 +18,17 @@
                 </material>
             </visual>
+            <collision>
+                <!-- 沿着自己几何中心的偏移和旋转 -->
+                <origin xyz="0.0 0.0 0.0" rpy="0.0 0.0 0.0"/>
+                <!-- 几何形状 -->
+                <geometry>
+                    <box size="0.02 0.10 0.02"/>
+                </geometry>
+                <!-- 材质描述 -->
+                <material name="black">
+                    <color rgba="0.0 0.0 0.0 0.5"/>
+                </material>
+            </collision>
+        <xacro:box_inertia m="0.1" w="0.02" h="0.10" d="0.02"/>
         </link>
         <!-- 机器人关节，用于组合部件 -->

File: robot/src/cerbers/urdf/cerbers/sensor/imu.urdf.xacro (robot description, xacro)
@@ -1,4 +1,5 @@
 <?xml version="1.0"?>
 <robot xmlns:xacro="http://www.ros.org/wiki/xacro">
+<xacro:include filename="$(find cerbers)/urdf/cerbers/common_inertial.xacro"/>
     <xacro:macro name="imu_xacro" params="xyz">
         <!-- 机器人的IMU，惯性测量传感器 -->
@@ -17,4 +18,17 @@
                 </material>
             </visual>
+            <collision>
+                <!-- 沿着自己几何中心的偏移和旋转 -->
+                <origin xyz="0.0 0.0 0.0" rpy="0.0 0.0 0.0"/>
+                <!-- 几何形状 -->
+                <geometry>
+                    <box size="0.02 0.02 0.02"/>
+                </geometry>
+                <!-- 材质描述 -->
+                <material name="black">
+                    <color rgba="0.0 0.0 0.0 0.5"/>
+                </material>
+            </collision>
+        <xacro:box_inertia m="0.05" w="0.02" h="0.02" d="0.02"/>
         </link>
         <!-- 机器人关节，用于组合部件 -->

File: robot/src/cerbers/urdf/cerbers/sensor/laser.urdf.xacro (robot description, xacro)
@@ -1,4 +1,5 @@
 <?xml version="1.0"?>
 <robot xmlns:xacro="http://www.ros.org/wiki/xacro">
+<xacro:include filename="$(find cerbers)/urdf/cerbers/common_inertial.xacro"/>
     <xacro:macro name="laser_xacro" params="xyz">
         <!-- 雷达支撑杆 -->
@@ -17,4 +18,17 @@
                 </material>
             </visual>
+            <collision>
+                <!-- 沿着自己几何中心的偏移和旋转 -->
+                <origin xyz="0.0 0.0 0.0" rpy="0.0 0.0 0.0"/>
+                <!-- 几何形状 -->
+                <geometry>
+                    <cylinder radius="0.01" length="0.10"/>
+                </geometry>
+                <!-- 材质描述 -->
+                <material name="black">
+                    <color rgba="0.0 0.0 0.0 1.0"/>
+                </material>
+            </collision>
+            <xacro:cylinder_inertia m="0.05" r="0.01" h="0.10" />
         </link>
         <!-- 雷达 -->
@@ -33,4 +47,16 @@
                 </material>
             </visual>
+            <collision>
+                <origin xyz="0.0 0.0 0.0" rpy="0.0 0.0 0.0"/>
+                <!-- 几何形状 -->
+                <geometry>
+                    <cylinder radius="0.02" length="0.02"/>
+                </geometry>
+                <!-- 材质描述 -->
+                <material name="black">
+                    <color rgba="0.0 0.0 0.0 1.0"/>
+                </material>
+            </collision>
+            <xacro:cylinder_inertia m="0.10" r="0.02" h="0.02" />
         </link>
         <!-- 机器人关节，用于组合部件 -->
