Commit message: 完成gazebo仿真与接入

File: robot/src/cerbers/urdf/cerbers/actuator/caster.urdf.xacro (robot description, xacro)
@@ -39,4 +39,10 @@
             <axis xyz="0.0 0.0 0.0"/>
         </joint>
+        <gazebo reference="${caster_name}_link">
+            <mu1 value="0.0"/>
+            <mu2 value="0.0"/>
+            <kp value="1000000000.0"/>
+            <kd value="1.0"/>
+        </gazebo>
     </xacro:macro>
 </robot>

File: robot/src/cerbers/urdf/cerbers/actuator/wheel.urdf.xacro (robot description, xacro)
@@ -39,4 +39,10 @@
             <axis xyz="0.0 1.0 0.0"/>
         </joint>
+        <gazebo reference="${wheel_name}_link">
+            <mu1 value="20.0"/>
+            <mu2 value="20.0"/>
+            <kp value="1000000000.0"/>
+            <kd value="1.0"/>
+        </gazebo>
     </xacro:macro>
 </robot>

File: robot/src/cerbers/urdf/cerbers/cerbers.urdf.xacro (robot description, xacro)
@@ -10,4 +10,7 @@
 <xacro:include filename="actuator/wheel.urdf.xacro"/>
 <xacro:include filename="actuator/caster.urdf.xacro"/>
+<!-- 插件 -->
+ <xacro:include filename="plugins/gazebo_control_plugin.xacro"/>
+ <xacro:include filename="plugins/gazebo_sensor_plugin.xacro"/>
 <!-- 调用宏 -->
 <xacro:base_xacro length="0.12" radius="0.1" />
@@ -19,3 +22,5 @@
 <xacro:caster_xacro caster_name="front_caster" xyz="0.08 0.0 -0.076" />
 <xacro:caster_xacro caster_name="back_caster" xyz="-0.08 0.0 -0.076" />
+<xacro:gazebo_control_plugin />
+<xacro:gazebo_sensor_plugin />
 </robot>

File: robot/src/cerbers/urdf/cerbers/sensor/camera.urdf.xacro (robot description, xacro)
@@ -32,4 +32,6 @@
         <xacro:box_inertia m="0.1" w="0.02" h="0.10" d="0.02"/>
         </link>
+        <link name="camera_optical_link">
+        </link>
         <!-- 机器人关节，用于组合部件 -->
         <joint name="camera_joint" type="fixed">
@@ -38,4 +40,10 @@
             <child link="camera_link"/>
         </joint>
+        <!-- 机器人关节，用于组合部件 -->
+        <joint name="camera_optical_joint" type="fixed">
+            <origin xyz="0 0 0" rpy="${-pi/2} 0.0 ${-pi/2}"/>
+            <parent link="camera_link"/>
+            <child link="camera_optical_link"/>
+        </joint>
     </xacro:macro>
 </robot>

File: robot/src/cerbers/urdf/cerbers/sensor/laser.urdf.xacro (robot description, xacro)
@@ -71,4 +71,10 @@
             <child link="laser_cylinder_link"/>
         </joint>
+        <gazebo reference="laser_cylinder_link">
+            <material>Gazebo/Black</material>
+        </gazebo>
+        <gazebo reference="laser_link">
+            <material>Gazebo/Black</material>
+        </gazebo>
     </xacro:macro>
 </robot>
